File: PCB/servo_driver/servo_driver.kicad_pcb (KiCad board)
At the start: 2 copper layers, 89 x 80.5 mm, 42 parts, among them J1 Conn_01x06, J2 Conn_01x02, J3 Conn_01x20, J4 Conn_01x20, J5 Conn_01x20, J6 Conn_01x20

Commit message: Hardware Update
Parts:
- added J7: Conn_01x03, Connector_JST:JST_PH_B3B-PH-K_1x03_P2.00mm_Vertical, F.Cu at (153.9, 109.2)
- J1: value Conn_01x06 -> Conn_01x03; footprint Connector_JST:JST_PH_S6B-PH-K_1x06_P2.00mm_Horizontal -> Connector_JST:JST_PH_B3B-PH-K_1x03_P2.00mm_Vertical; moved to F.Cu
- moved J1 46.2 mm to (153.9, 58.0)
- moved J2 37.3 mm to (116.5, 77.2)
- moved Vin+1 17.3 mm to (115.5, 124.9)
- moved Vout+1 16.7 mm to (131.6, 125.0)
- moved Vin-1 16.6 mm to (115.5, 114.9)
- moved Vout-1 16.0 mm to (131.6, 115.1)
- moved Vin+2 15.1 mm to (115.5, 109.4)
- moved C1 14.8 mm to (138.0, 118.9)
- moved C2 14.8 mm to (138.0, 106.4)
- moved Servo1 14.8 mm to (145.5, 121.4)
- moved Servo2 14.8 mm to (145.5, 108.9)
- moved Vin-2 14.5 mm to (115.5, 99.4)
- moved Vout+2 14.4 mm to (131.6, 109.5)
- moved Vout-2 13.8 mm to (131.6, 99.6)
- moved Vin-6 11.0 mm to (115.8, 37.3)
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Connections:
- Servo1 pad 1: Net-(J1-Pin_1) -> Net-(J7-Pin_1)
- Servo2 pad 1: Net-(J1-Pin_2) -> Net-(J7-Pin_2)
- Servo3 pad 1: Net-(J1-Pin_3) -> Net-(J7-Pin_3)
- Servo4 pad 1: Net-(J1-Pin_4) -> Net-(J1-Pin_1)
- Servo5 pad 1: Net-(J1-Pin_5) -> Net-(J1-Pin_2)
- Servo6 pad 1: Net-(J1-Pin_6) -> Net-(J1-Pin_3)
Routing:
- net Net-(J1-Pin_6): track 65.4 -> 0.00 mm
- net Net-(J1-Pin_5): track 55.7 -> 0.00 mm
- net Net-(J1-Pin_1): track 54.4 -> 0.00 mm
- net Net-(J1-Pin_2): track 45.3 -> 0.00 mm
- net Net-(J1-Pin_4): track 44.7 -> 0.00 mm
- net Net-(J1-Pin_3): track 37.8 -> 0.00 mm
- net Net-(Servo6-Pin_2): track 15.2 -> 7.52 mm
- net Net-(Servo4-Pin_2): track 15.2 -> 7.52 mm
- net Net-(Servo3-Pin_2): track 15.2 -> 7.52 mm
- net Net-(Servo2-Pin_2): track 15.2 -> 7.52 mm
- net Net-(Servo1-Pin_2): track 15.2 -> 7.52 mm
- net Net-(Servo5-Pin_2): track 14.8 -> 7.52 mm
- net Net-(Servo6-Pin_3): track 14.6 -> 7.53 mm
- net Net-(Servo5-Pin_3): track 14.6 -> 7.53 mm
- net Net-(Servo4-Pin_3): track 14.6 -> 7.53 mm
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- removed copper zone on B.Cu, net Bat+
- removed copper zone on B.Cu, net Bat-
- removed copper zone on F.Cu, net Bat-
Other:
- board size 89 x 80.5 mm -> 89 x 92.5 mm
